File: can1.kicad_sch (KiCad schematic)
At the start: 1 part, among them U1 TJA1042T-3

Commit message: finalize CAN1
Parts:
- added C1: C, Capacitor_SMD:C_1206_3216Metric_Pad1.33x1.80mm_HandSolder, symbol Device:C
- added C2, C3: 47nF, Capacitor_SMD:C_1206_3216Metric_Pad1.33x1.80mm_HandSolder, symbol Device:C
- added R1, R2, R3: R, Resistor_SMD:R_1206_3216Metric_Pad1.30x1.75mm_HandSolder, symbol Device:R
Connections:
- net +3V3: now also C2.1
- net +5V: now also C3.1
- net CAN1_H: now also R1.1
- net CAN1_L: now also R2.1
- net GND: now also C1.2, C2.2, C3.2, R3.2
- net CAN1_STB: now reaches U1.8 (STB)
- net CAN1_STB: now also R3.1
- new net: C1.1, R1.2, R2.2
