File: uarts.kicad_sch (KiCad schematic)
At the start: 2 parts

Commit message: place CNs correctly (?)
Parts:
- renumbered DeviceUART to DeviceUART1, RoutedUART to RoutedUART1
Changed lines of the file:
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@@
+	(wire
+		(pts
+			(xy 124.46 71.12) (xy 137.16 71.12)
+		)
+		(stroke
+			(width 0)
+			(type default)
+		)
+	)
+	(wire
+		(pts
+			(xy 66.04 78.74) (xy 74.93 78.74)
+		)
+		(stroke
+			(width 0)
+			(type default)
+		)
+	)
+	(wire
+		(pts
+			(xy 66.04 83.82) (xy 74.93 83.82)
+		)
+		(stroke
+			(width 0)
+			(type default)
+		)
+	)
+	(wire
+		(pts
+			(xy 72.39 76.2) (xy 74.93 76.2)
+		)
+		(stroke
+			(width 0)
+			(type default)
+		)
+	)
+	(wire
+		(pts
+			(xy 66.04 66.04) (xy 74.93 66.04)
+		)
+		(stroke
+			(width 0)
+			(type default)
+		)
+	)
+	(wire
+		(pts
+			(xy 134.62 76.2) (xy 137.16 76.2)
+		)
+		(stroke
+			(width 0)
+			(type default)
+		)
+	)
 	(wire
 		(pts
@@
 	(wire
 		(pts
+			(xy 66.04 71.12) (xy 74.93 71.12)
+		)
+		(stroke
+			(width 0)
+			(type default)
+		)
+	)
+	(wire
+		(pts
+			(xy 124.46 73.66) (xy 137.16 73.66)
+		)
+		(stroke
+			(width 0)
+			(type default)
+		)
+	)
+	(wire
+		(pts
+			(xy 66.04 86.36) (xy 74.93 86.36)
+		)
+		(stroke
+			(width 0)
+			(type default)
+		)
+	)
+	(wire
+		(pts
 			(xy 124.46 68.58) (xy 137.16 68.58)
 		)
@@
 	(wire
 		(pts
-			(xy 124.46 73.66) (xy 137.16 73.66)
-		)
-		(stroke
-			(width 0)
-			(type default)
-		)
-	)
-	(wire
-		(pts
-			(xy 72.39 76.2) (xy 74.93 76.2)
+			(xy 66.04 68.58) (xy 74.93 68.58)
 		)
 		(stroke
@@
 	(wire
 		(pts
-			(xy 66.04 78.74) (xy 74.93 78.74)
+			(xy 66.04 81.28) (xy 74.93 81.28)
+		)
+		(stroke
+			(width 0)
+			(type default)
+		)
+	)
+	(wire
+		(pts
+			(xy 124.46 78.74) (xy 137.16 78.74)
+		)
+		(stroke
+			(width 0)
+			(type default)
+		)
+	)
+	(wire
+		(pts
+			(xy 66.04 73.66) (xy 74.93 73.66)
 		)
 		(stroke
@@
 	(wire
 		(pts
-			(xy 124.46 71.12) (xy 137.16 71.12)
-		)
-		(stroke
-			(width 0)
-			(type default)
-		)
-	)
-	(wire
-		(pts
-			(xy 134.62 76.2) (xy 137.16 76.2)
-		)
-		(stroke
-			(width 0)
-			(type default)
-		)
-	)
-	(wire
-		(pts
-			(xy 66.04 86.36) (xy 74.93 86.36)
-		)
-		(stroke
-			(width 0)
-			(type default)
-		)
-	)
-	(wire
-		(pts
-			(xy 66.04 83.82) (xy 74.93 83.82)
-		)
-		(stroke
-			(width 0)
-			(type default)
-		)
-	)
-	(wire
-		(pts
 			(xy 124.46 86.36) (xy 137.16 86.36)
-		)
-		(stroke
-			(width 0)
-			(type default)
-		)
-	)
-	(wire
-		(pts
-			(xy 66.04 81.28) (xy 74.93 81.28)
-		)
-		(stroke
-			(width 0)
-			(type default)
-		)
-	)
-	(wire
-		(pts
-			(xy 66.04 73.66) (xy 74.93 73.66)
-		)
-		(stroke
-			(width 0)
-			(type default)
-		)
-	)
-	(wire
-		(pts
-			(xy 66.04 66.04) (xy 74.93 66.04)
-		)
-		(stroke
-			(width 0)
-			(type default)
-		)
-	)
-	(wire
-		(pts
-			(xy 124.46 78.74) (xy 137.16 78.74)
-		)
-		(stroke
-			(width 0)
-			(type default)
-		)
-	)
-	(wire
-		(pts
-			(xy 66.04 71.12) (xy 74.93 71.12)
-		)
-		(stroke
-			(width 0)
-			(type default)
-		)
-	)
-	(wire
-		(pts
-			(xy 66.04 68.58) (xy 74.93 68.58)
 		)
 		(stroke
@@
 		(dnp no)
 		(fields_autoplaced yes)
-		(property "Reference" "DeviceUART"
+		(property "Reference" "DeviceUART1"
 			(at 87.63 74.9299 0)
 			(effects
@@
 			(project "sample"
 				(path "/b24c09df-2e49-4fc3-a45d-ba0b1ff2d257/f41f9e10-c9db-46df-9898-e9f35bc46669"
-					(reference "DeviceUART")
+					(reference "DeviceUART1")
 					(unit 1)
 				)
@@
 		(dnp no)
 		(fields_autoplaced yes)
-		(property "Reference" "RoutedUART"
+		(property "Reference" "RoutedUART1"
 			(at 149.86 74.9299 0)
 			(effects
@@
 			(project "sample"
 				(path "/b24c09df-2e49-4fc3-a45d-ba0b1ff2d257/f41f9e10-c9db-46df-9898-e9f35bc46669"
-					(reference "RoutedUART")
+					(reference "RoutedUART1")
 					(unit 1)
 				)

Commit message: uarts routed
Connections:
- net UART4_RX: now also DeviceUART1.5; no longer RoutedUART1.1
- net UART4_TX: now also DeviceUART1.9; no longer RoutedUART1.6
- net UART7_RX: now also DeviceUART1.6; no longer RoutedUART1.8
- net UART7_TX: now also DeviceUART1.1; no longer RoutedUART1.4
- net UART9_RX: now also DeviceUART1.4; no longer RoutedUART1.9
- net UART9_TX: now also DeviceUART1.8; no longer RoutedUART1.5
- net USART10_RX: now also RoutedUART1.9; no longer DeviceUART1.5
- net USART10_TX: now also RoutedUART1.5; no longer DeviceUART1.9
- net USART2_RX: now also RoutedUART1.8; no longer DeviceUART1.6
- net USART2_TX: now also RoutedUART1.4; no longer DeviceUART1.1
- net USART6_RX: now also RoutedUART1.1; no longer DeviceUART1.4
- net USART6_TX: now also RoutedUART1.6; no longer DeviceUART1.8
Other:
- moved on the sheet: RoutedUART1
